Commit message: correct position of thrusters and add dummy inertia values

File: src/models/urdf/auv_model.urdf (robot description, URDF)
Before this commit: robot auv, 5 links, 4 joints
Links:
- link back_thruster: mass 0.0 -> 0.5
- link base_link: mass 0.0 -> 1.0
- link front_thruster: mass 0.0 -> 0.5
- link left_thruster: mass 0.0 -> 0.5
- link right_thruster: mass 0.0 -> 0.5
