Commit message: add camera link and plugin

File: src/models/urdf/auv_model.xacro (robot description, xacro)
@@ -97,4 +97,25 @@
         </collision>
     </link>
+    <link name="camera_front">
+        <inertial>
+            <origin xyz="0.0 0.0 0.0" rpy="0.0 0.0 0.0"/>
+            <mass value="1.0"/>
+            <inertia ixx="1.0" ixy="0.0" ixz="0.0" iyy="1.0" iyz="0.0" izz="1.0"/>
+        </inertial>
+        <visual name="">
+            <origin xyz="0.0 0.0 0.0" rpy="0.0 0.0 0.0"/>
+            <geometry>
+                <box size="0.01 0.01 0.01"/>
+            </geometry>
+        </visual>
+        <collision>
+            <origin xyz="0.0 0.0 0.0" rpy="0.0 0.0 0.0"/>
+            <geometry>
+                <box size="0.01 0.01 0.01"/>
+            </geometry>
+        </collision>
+    </link>
+    <link name="frontCam_optical">
+    </link>
     <joint name="leftThruster_baseLink" type="fixed">
         <origin xyz="0.0 -0.18 0.0" rpy="0.0 0.0 0.0"/>
@@ -125,3 +146,17 @@
         <limit lower="0.0" upper="0.0" effort="0.0" velocity="0.0"/>
     </joint>
+    <joint name="frontCamera_joint" type="fixed">
+        <origin xyz="0.3 0. 0.06" rpy="0.0 0.0 0.0"/>
+        <parent link="base_link"/>
+        <child link="camera_front"/>
+        <axis xyz="0.0 0.0 0.0"/>
+        <limit lower="0.0" upper="0.0" effort="0.0" velocity="0.0"/>
+    </joint>
+    <joint name="frontCamera_opticalJoint" type="fixed">
+        <origin xyz="0.0 0.0 0.0" rpy="-1.5707 0 -1.5707"/>
+        <parent link="camera_front"/>
+        <child link="frontCam_optical"/>
+        <axis xyz="0.0 0.0 0.0"/>
+        <limit lower="0.0" upper="0.0" effort="0.0" velocity="0.0"/>
+    </joint>
 </robot>

Commit message: correct gazebo launch file and

File: src/models/urdf/auv_model.xacro (robot description, xacro)
@@ -116,5 +116,5 @@
         </collision>
     </link>
-    <link name="frontCam_optical">
+    <link name="camera_front_optical">
     </link>
     <joint name="leftThruster_baseLink" type="fixed">
@@ -156,5 +156,5 @@
         <origin xyz="0.0 0.0 0.0" rpy="-1.5707 0 -1.5707"/>
         <parent link="camera_front"/>
-        <child link="frontCam_optical"/>
+        <child link="camera_front_optical"/>
         <axis xyz="0.0 0.0 0.0"/>
         <limit lower="0.0" upper="0.0" effort="0.0" velocity="0.0"/>

Commit message: add imu link and  bottom camera

File: src/models/urdf/auv_model.xacro (robot description, xacro)
@@ -21,4 +21,26 @@
         </collision>
     </link>
+<<<<<<< HEAD
+    <link name="imu_link">
+        <inertial>
+            <origin xyz="0.0 0.0 0.0" rpy="0.0 0.0 0.0"/>
+            <mass value="1.0"/>
+            <inertia ixx="1.0" ixy="0.0" ixz="0.0" iyy="1.0" iyz="0.0" izz="1.0"/>
+        </inertial>
+        <visual name="">
+            <origin xyz="0.0 0.0 0.0" rpy="0.0 0.0 0.0"/>
+            <geometry>
+                <box size="0.01 0.01 0.01"/>
+            </geometry>
+        </visual>
+        <collision>
+            <origin xyz="0.0 0.0 0.0" rpy="0.0 0.0 0.0"/>
+            <geometry>
+                <box size="0.01 0.01 0.01"/>
+            </geometry>
+        </collision>
+    </link>
+=======
+>>>>>>> 6df93dd37ae20203b9764f8cb4ff4d51d771fc73
     <link name="right_thruster">
         <inertial>
@@ -116,6 +138,40 @@
         </collision>
     </link>
+<<<<<<< HEAD
+     <link name="camera_bottom">
+        <inertial>
+            <origin xyz="0.0 0.0 0.0" rpy="0.0 0.0 0.0"/>
+            <mass value="1.0"/>
+            <inertia ixx="1.0" ixy="0.0" ixz="0.0" iyy="1.0" iyz="0.0" izz="1.0"/>
+        </inertial>
+        <visual name="">
+            <origin xyz="0.0 0.0 0.0" rpy="0.0 0.0 0.0"/>
+            <geometry>
+                <box size="0.01 0.01 0.01"/>
+            </geometry>
+        </visual>
+        <collision>
+            <origin xyz="0.0 0.0 0.0" rpy="0.0 0.0 0.0"/>
+            <geometry>
+                <box size="0.01 0.01 0.01"/>
+            </geometry>
+        </collision>
+    </link>
+=======
+>>>>>>> 6df93dd37ae20203b9764f8cb4ff4d51d771fc73
     <link name="camera_front_optical">
     </link>
+<<<<<<< HEAD
+    <link name ="camera_bottom_optical">
+    </link>
+    <joint name="imu_baseLink" type="fixed">
+        <origin xyz="0.0 0.0 0.0" rpy="0.0 0.0 0.0"/>
+        <parent link="base_link"/>
+        <child link="imu_link"/>
+        <axis xyz="0.0 0.0 0.0"/>
+        <limit lower="0.0" upper="0.0" effort="0.0" velocity="0.0"/>
+    </joint>
+=======
+>>>>>>> 6df93dd37ae20203b9764f8cb4ff4d51d771fc73
     <joint name="leftThruster_baseLink" type="fixed">
         <origin xyz="0.0 -0.18 0.0" rpy="0.0 0.0 0.0"/>
@@ -160,3 +216,20 @@
         <limit lower="0.0" upper="0.0" effort="0.0" velocity="0.0"/>
     </joint>
+<<<<<<< HEAD
+    <joint name="bottomCamera_joint" type="fixed">
+        <origin xyz="0.0 0.0 -0.06" rpy="0.0 -1.5707 0.0"/>
+        <parent link="base_link"/>
+        <child link="camera_bottom"/>
+        <axis xyz="0.0 0.0 0.0"/>
+        <limit lower="0.0" upper="0.0" effort="0.0" velocity="0.0"/>
+    </joint>
+    <joint name="bottomCamera_opticalJoint" type="fixed">
+        <origin xyz="0.0 0.0 0.0" rpy="-1.5707 0 -1.5707"/>
+        <parent link="camera_bottom"/>
+        <child link="camera_bottom_optical"/>
+        <axis xyz="0.0 0.0 0.0"/>
+        <limit lower="0.0" upper="0.0" effort="0.0" velocity="0.0"/>
+    </joint>
+=======
+>>>>>>> 6df93dd37ae20203b9764f8cb4ff4d51d771fc73
 </robot>
